File: LED_Tile_Controller.kicad_pcb (KiCad board)
At the start: 4 copper layers, 88 x 36.6 mm, 49 parts, among them J1 AVX 009159008061816, J4 Conn_01x04, J5 USB_C_Receptacle_USB2.0, J6 Stemma/QT, J7 Conn_01x02, J8 Conn_01x07, J9 Conn_02x03_Odd_Even, SW1 SW_Push, SW2 SW_Push, U2 ESP32-C3-MINI-1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

Commit message: led tile controller working nicely :-)
Parts:
- removed C9: 1nF 10V, Capacitor_SMD:C_0402_1005Metric
- added C4: 100nF 10V, Capacitor_SMD:C_0402_1005Metric, F.Cu at (145.8, 75.2)
- added LO1: Robo_Logo, runger:Robo_logo2, B.Cu at (117.1, 56.5)
- added R14: 10k, Resistor_SMD:R_0402_1005Metric, F.Cu at (156.0, 76.2)
- added R15: 20k, Resistor_SMD:R_0402_1005Metric, F.Cu at (154.5, 75.1)
- added R16: 10k, Resistor_SMD:R_0402_1005Metric, F.Cu at (146.8, 76.2)
- U3: value ACS725 -> CC6900SO-5A
Connections:
- C11 pad 2: VDD -> +5V
- U2 pad 6: /VIOUT -> Net-(C4-Pad2)
- U3 pad 6: Net-(C9-Pad2) -> unconnected-(U3-Pad6)
- U3 pad 7: /VIOUT -> Net-(R14-Pad2)
- U3 pad 8: VDD -> +5V
Routing:
- net /VIOUT: track 18.9 -> 8.81 mm
- net Net-(R14-Pad2): track 0.00 -> 4.99 mm
- net Net-(C4-Pad2): track 0.00 -> 4.87 mm
- net +5V: track 47.2 -> 51.0 mm
- net VDD: track 118.0 -> 114.7 mm
- net Net-(C9-Pad2): track 1.86 -> 0.00 mm
- net GND: track 86.0 -> 87.7 mm
Other:
- board text added: "ESP32-C3"
- board text added: "LED Tile Controller"
- board text added: "©2023 runger"
